File: Tesla_rev_2/MCU.kicad_sch (KiCad schematic)
At the start: 3 parts, among them U9 ESP32-WROOM-32D

Commit message: Netclasses, part Nums, LPF adjust
Parts:
- renumbered C44 to C45, C45 to C46
Other:
- title: (none) -> Tesla sextant BT
Changed lines of the file:
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@@
 	(generator_version "9.0")
 	(paper "A4")
+	(title_block
+		(title "Tesla sextant BT")
+		(date "2025-11-30")
+		(rev "2.1")
+	)
 	(junction
 		(at 146.05 62.865)
@@
 		(dnp no)
 		(fields_autoplaced yes)
-		(property "Reference" "#PWR0106"
+		(property "Reference" "#PWR?"
 			(at 146.05 46.99 0)
 			(effects
@@
 			(project "Tesla_sextant_BT"
 				(path "/8e7bde30-d14b-44a7-a566-3173755ec64c/9ff7eca1-18ea-42ec-8229-18347a2ef5b0"
-					(reference "#PWR0106")
+					(reference "#PWR?")
 					(unit 1)
 				)
@@
 		(on_board yes)
 		(dnp no)
-		(property "Reference" "#PWR0108"
+		(property "Reference" "#PWR?"
 			(at 138.43 69.215 0)
 			(effects
@@
 			(project "Tesla_sextant_BT"
 				(path "/8e7bde30-d14b-44a7-a566-3173755ec64c/9ff7eca1-18ea-42ec-8229-18347a2ef5b0"
-					(reference "#PWR0108")
+					(reference "#PWR?")
 					(unit 1)
 				)
@@
 		(dnp no)
 		(fields_autoplaced yes)
-		(property "Reference" "#PWR0109"
+		(property "Reference" "#PWR?"
 			(at 146.05 142.24 0)
 			(effects
@@
 			(project "Tesla_sextant_BT"
 				(path "/8e7bde30-d14b-44a7-a566-3173755ec64c/9ff7eca1-18ea-42ec-8229-18347a2ef5b0"
-					(reference "#PWR0109")
+					(reference "#PWR?")
 					(unit 1)
 				)
@@
 		(dnp no)
 		(fields_autoplaced yes)
-		(property "Reference" "C45"
+		(property "Reference" "C46"
 			(at 142.24 55.88 90)
 			(effects
@@
 			(project "Tesla_sextant_BT"
 				(path "/8e7bde30-d14b-44a7-a566-3173755ec64c/9ff7eca1-18ea-42ec-8229-18347a2ef5b0"
-					(reference "C45")
+					(reference "C46")
 					(unit 1)
 				)
@@
 		(dnp no)
 		(fields_autoplaced yes)
-		(property "Reference" "C44"
+		(property "Reference" "C45"
 			(at 142.24 43.815 90)
 			(effects
@@
 			(project "Tesla_sextant_BT"
 				(path "/8e7bde30-d14b-44a7-a566-3173755ec64c/9ff7eca1-18ea-42ec-8229-18347a2ef5b0"
-					(reference "C44")
+					(reference "C45")
 					(unit 1)
 				)
@@
 		(dnp no)
 		(fields_autoplaced yes)
-		(property "Reference" "#PWR0107"
+		(property "Reference" "#PWR?"
 			(at 138.43 57.785 0)
 			(effects
@@
 			(project "Tesla_sextant_BT"
 				(path "/8e7bde30-d14b-44a7-a566-3173755ec64c/9ff7eca1-18ea-42ec-8229-18347a2ef5b0"
-					(reference "#PWR0107")
+					(reference "#PWR?")
 					(unit 1)
 				)
