File: Tesla_rev_2/Tesla_sextant_BT.kicad_sch (KiCad schematic)
At the start: 37 parts, among them J1 Conn_01x07, J2 Conn_01x07, J3 Conn_01x02, J4 Conn_01x03, J5 Conn_01x03, J6 Conn_01x02, J7 Conn_01x05, J8 Conn_Coaxial, J9 Conn_01x02, U1 LA1185, Y1 Crystal

Commit message: Netclasses, part Nums, LPF adjust
Parts:
- removed C2: 10uF, Capacitor_SMD:CP_Elec_6.3x7.7, symbol Device:C_Polarized
- added C47: 10uF, symbol Device:C_Polarized
- renumbered C10 to C1, C9 to C10, C12 to C11, C6 to C12, C1 to C2, C4 to C3, C7 to C4, C8 to C6, C11 to C7, C3 to C9, J4 to J2, J8 to J3, J2 to J4, J7 to J6, J6 to J7, J9 to J8, J3 to J9
Connections:
- net +5V: now also C47.1
- net GND: now also C47.2
- net DAC_AMP/VO+ renamed DAC_AMP/AUDIO_O+
- net DAC_AMP/VO- renamed DAC_AMP/AUDIO_O-
Other:
- sheet DAC_AMP ports: added AUDIO_O+, AUDIO_O-; removed VO+, VO-
- note added: "87,5 - 108MHz to 65,5 - 74 MHz convertor"
