File: Tesla_rev_2/DAC_AMP.kicad_sch (KiCad schematic)
At the start: 37 parts, among them K1 G6EU, Q1 BC817, U2 PCM5102A, U3 OPA2342, U4 TPA0211

Commit message: Board ready for manufacturing, no more changes to either KiCad projects
Parts:
- removed C14: 100nF, Capacitor_SMD:C_0805_2012Metric, symbol Device:C
- removed C17: 10uF, Capacitor_SMD:C_0805_2012Metric, symbol Device:C
- removed D3: B220, Diode_SMD:D_SMB, symbol Diode:B220
- removed K1: G6EU, Relay_THT:Relay_SPDT_Omron_G6E, symbol Relay:G6EU
- removed R14: 7.5K, Capacitor_SMD:C_0805_2012Metric, symbol Device:R
- removed R17: 1K, Capacitor_SMD:C_0805_2012Metric, symbol Device:R
- removed R18: TBD, Capacitor_SMD:C_0805_2012Metric, symbol Device:R
- removed R19, R20: 100K, Capacitor_SMD:C_0805_2012Metric, symbol Device:R
- removed TP3: TestPoint, TestPoint:TestPoint_Pad_D2.5mm, symbol Connector:TestPoint
- removed U3: OPA2342, Package_SO:SOIC-8_3.9x4.9mm_P1.27mm, symbol Tesla_sextant_BT_Library:OPA2342
- added D3: B240, Diode_SMD:D_SMB, symbol Diode:B240
- added K1: G5V-1, Relay_THT:Relay_SPDT_Omron_G5V-1, symbol Relay:G5V-1
- R10, R11, R15, R16, R8, R9: footprint Capacitor_SMD:C_0805_2012Metric -> Resistor_SMD:R_0805_2012Metric
Connections:
- net +5V: now also D3.1 (K), K1.2
- net AUD_AMP: now also K1.5, K1.6
- net AUD_DAC_MIX: now also K1.10
- net AUD_RADIO: now also K1.1
- net REL_PULLD: now also D3.2 (A), K1.9
Other:
- note removed: "Buffer + bias"
- note removed: "Optional gain setting"
- moved on the sheet: C10, C11, C12, C13, C15, C16, C3, C4, C41, C5, C6, C7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

Commit message: Final Project Commit
Parts:
- C41: now fitted
