File: Tesla_rev_2/POWER.kicad_sch (KiCad schematic)
At the start: 40 parts, among them J6 USB_C_Receptacle_USB2.0_16P, J7 Conn_01x03, U5 USBLC6-2SC6, U6 AP63203WU, U7 LD1117STR

Commit message: Board ready for manufacturing, no more changes to either KiCad projects
Parts:
- R22, R23, R25, R26: footprint Capacitor_SMD:C_0805_2012Metric -> Resistor_SMD:R_0805_2012Metric
Changed lines of the file:
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@@
 	(title_block
 		(title "Tesla sextant BT POWER")
-		(date "2026-02-10")
-		(rev "2.3")
+		(date "2026-02-24")
+		(rev "2.4")
 	)
 	(text "Uout = ~10V\nUout = 1.25 * (1 + (R2/R1))\n10 = 1.25 * (1 + (R2/120))\nR2 = 840 => 820\n"
@@
 			)
 		)
-		(property "Footprint" "Capacitor_SMD:C_0805_2012Metric"
+		(property "Footprint" "Resistor_SMD:R_0805_2012Metric"
 			(at 228.727 74.295 90)
 			(effects
@@
 			)
 		)
-		(property "Footprint" "Capacitor_SMD:C_0805_2012Metric"
+		(property "Footprint" "Resistor_SMD:R_0805_2012Metric"
 			(at 237.617 74.295 90)
 			(effects
@@
 			)
 		)
-		(property "Footprint" "Capacitor_SMD:C_0805_2012Metric"
+		(property "Footprint" "Resistor_SMD:R_0805_2012Metric"
 			(at 69.342 138.43 90)
 			(effects
@@
 			)
 		)
-		(property "Footprint" "Capacitor_SMD:C_0805_2012Metric"
+		(property "Footprint" "Resistor_SMD:R_0805_2012Metric"
 			(at 69.342 146.05 90)
 			(effects
