File: Tesla_rev_2/Tesla_sextant_BT.kicad_pcb (KiCad board)
At the start: 4 copper layers, 100 x 100 mm, 130 parts, among them J1 Conn_01x05, J2 Conn_01x02, J3 Conn_01x05, J4 Conn_01x02, J6 USB_C_Receptacle_USB2.0_16P, J7 Conn_01x03, J8 Conn_01x02, J9 Conn_01x02, K1 G6EU, Q1 BC817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

Commit message: changes with BOM, minor fixes
Parts:
- moved L5 0.05 mm to (123.5, 139.2)
- moved C35 0.05 mm to (127.8, 140.2)
Routing:
- net +3.3V: track 313.6 -> 317.0 mm
- net GND: vias 203 -> 204
Other:
- rule pad_to_mask_clearance: 0.0762 -> 0.05
- board text added: "C32"
- board text added: "Rev. 2.2 | 2026-02-22"
- board text removed: "Rev. 2.1 | 2026-02-10"

Commit message: Board ready for manufacturing, no more changes to either KiCad projects
Parts:
- removed C14: 100nF, Capacitor_SMD:C_0805_2012Metric
- removed C17: 10uF, Capacitor_SMD:C_0805_2012Metric
- removed C43: 2.2nF, Capacitor_SMD:C_0603_1608Metric
- removed R14: 7.5K, Capacitor_SMD:C_0805_2012Metric
- removed R17: 1K, Capacitor_SMD:C_0805_2012Metric
- removed R18: TBD, Capacitor_SMD:C_0805_2012Metric
- removed R19, R20: 100K, Capacitor_SMD:C_0805_2012Metric
- removed TP3: TestPoint, TestPoint:TestPoint_Pad_D2.5mm
- removed U3: OPA2342, Package_SO:SOIC-8_3.9x4.9mm_P1.27mm
- added R34: 75, Resistor_SMD:R_0805_2012Metric, F.Cu at (162.3, 139.3)
- C31: value 5.6pF -> 5pF
- C32: value 4.7pF -> 130pF
- C33: value 470pF -> 100nF
- C34: value 220pF -> 5pF
- C35: value TBD -> 5pF; footprint Capacitor_SMD:C_0805_2012Metric -> Capacitor_SMD:C_0603_1608Metric
- C36: value 100nF -> 510pF; footprint Capacitor_SMD:C_0805_2012Metric -> Capacitor_SMD:C_0603_1608Metric
- C39: value 2.2nF -> 44pF
- D3: value B220 -> B240
- K1: value G6EU -> G5V-1; footprint Relay_THT:Relay_SPDT_Omron_G6E -> Relay_THT:Relay_SPDT_Omron_G5V-1
- L3: value 870nF -> 1uH; footprint Inductor_SMD:L_0805_2012Metric -> Inductor_SMD:L_0603_1608Metric
- L4: value 1.3uF -> 40nH; footprint Inductor_SMD:L_0805_2012Metric -> Inductor_SMD:L_0603_1608Metric
- L5: value TBD -> 430nH
- L6: value 12nH -> MABAES0060; footprint Inductor_SMD:L_0603_1608Metric -> Tesla_Library:SM-22
- L7: value 20nH -> MABAES0060; footprint Inductor_SMD:L_0603_1608Metric -> Tesla_Library:SM-22
- L8: value 18nH -> 900nH
- R1, R10, R11, R15, R16, R2, R22, R23, R25, R26, R28, R3, R30, R31, R32, R4, R5, R6, R7, R8, R9: footprint Capacitor_SMD:C_0805_2012Metric -> Resistor_SMD:R_0805_2012Metric
- R27, R33: value 50 -> 75; footprint Capacitor_SMD:C_0805_2012Metric -> Resistor_SMD:R_0805_2012Metric
- R29: value 50 -> 200; footprint Capacitor_SMD:C_0805_2012Metric -> Resistor_SMD:R_0805_2012Metric
- moved L7 36.2 mm to (126.4, 138.2)
- moved C34 32.8 mm to (128.0, 139.8), turned to 0 degrees
- moved R29 27.5 mm to (138.8, 149.2), turned to 180 degrees
- moved R15 21.2 mm to (143.1, 116.8), turned to 90 degrees
- moved L6 18.1 mm to (171.1, 145.8), turned to 180 degrees
- moved Q1 15.5 mm to (144.1, 112.9), turned to 90 degrees
- moved C33 14.9 mm to (138.8, 142.0), turned to -90 degrees
- moved C36 13.8 mm to (141.3, 151.2), turned to 180 degrees
- moved D3 9.73 mm to (144.9, 106.3)
- moved C9 9.71 mm to (144.8, 100.5)
- moved J8 8.05 mm to (176.8, 147.5)
- moved U4 7.50 mm to (165.9, 115.9)
- moved C15 7.50 mm to (158.4, 111.8)
- moved C16 7.50 mm to (163.7, 119.5)
- moved R16 7.50 mm to (162.7, 111.8)
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Connections:
- net /freq_converter/IF_R1 renamed /freq_converter/IF_TERM
- net /freq_converter/LO_HPF renamed /freq_converter/LO_L1
- C31 pad 2: /freq_converter/IF_C1 -> /freq_converter/IF_C
- C32 pad 1: /freq_converter/IF_C3 -> GND
- C32 pad 2: /freq_converter/IF_FLT -> /freq_converter/IF_BPF
- C33 pad 1: GND -> /freq_converter/RF_IN-
- C33 pad 2: /freq_converter/IF_FLT -> GND
- C34 pad 1: GND -> /freq_converter/RF_T
- C34 pad 2: /freq_converter/IF_OUT -> /freq_converter/RF_Z
- C35 pad 1: GND -> /freq_converter/RF_Z
- C36 pad 1: GND -> Net-(C36-Pad1)
- C36 pad 2: /freq_converter/RF_IN- -> GND
- C39 pad 1: GND -> /freq_converter/LO_LPF
- J8 pad 1: /freq_converter/IF_OUT -> /freq_converter/IF_OUT+
- J8 pad 2: GND -> /freq_converter/IF_OUT-
- J9 pad 1: /freq_converter/RF_CONN -> /freq_converter/RF_CONN+
- J9 pad 2: GND -> /freq_converter/RF_CONN-
- K1 pad 1: +5V -> /DAC_AMP/AUD_RADIO
- K1 pad 10: /DAC_AMP/AUD_RADIO -> /DAC_AMP/AUD_DAC_MIX
- K1 pad 6: /DAC_AMP/REL_PULLD -> /DAC_AMP/AUD_AMP
- L3 pad 1: /freq_converter/IF_FLT -> /freq_converter/IF_C
- L3 pad 2: /freq_converter/IF_C1 -> /freq_converter/IF_BPF
- L4 pad 1: /freq_converter/IF_OUT -> /freq_converter/IF_BPF
- L4 pad 2: /freq_converter/IF_C3 -> GND
- L5 pad 1: /freq_converter/RF_IN+ -> /freq_converter/RF_Z
- L5 pad 2: /freq_converter/RF_CONN -> GND
- L6 pad 1: GND -> /freq_converter/IF_OUT+
- L6 pad 2: /freq_converter/IF_FLT -> GND
- L7 pad 1: /freq_converter/IF_OUT -> /freq_converter/RF_T
- L7 pad 2: GND -> unconnected-(L7-Pad2)
- L8 pad 1: /freq_converter/LO_OSC -> Net-(C36-Pad1)
- R29 pad 1: GND -> Net-(C36-Pad1)
- R29 pad 2: /freq_converter/IF_OUT -> /freq_converter/LO_OSC
Routing:
- net /AUDIO_SEL: track 32.3 -> 56.2 mm
- net /DAC_AMP/AUD_BUFF: track 19.9 -> 0.00 mm, vias 1 -> 0
- net +5V: track 141.5 -> 125.0 mm, vias 9 -> 8
- net /DAC_AMP/OP_AMP_BIAS: track 15.7 -> 0.00 mm
- net /DAC_AMP/AUD_AMP: track 23.6 -> 8.68 mm
- net /freq_converter/IF_OUT: track 14.9 -> 0.00 mm
- net /freq_converter/IF_OUT-: track 0.00 -> 13.6 mm
- net /freq_converter/IF_OUT+: track 0.00 -> 12.6 mm
- net /freq_converter/IF_BPF: track 0.00 -> 12.1 mm
- net /DAC_AMP/DIV_2.5V: track 11.6 -> 0.00 mm, vias 2 -> 0
- net /freq_converter/RF_CONN: track 8.72 -> 0.00 mm
- net /DAC_AMP/AUDIO_OUT-: track 18.6 -> 26.6 mm
- net /DAC_AMP/REL_PULLD: track 22.6 -> 14.7 mm
- net /freq_converter/RF_CONN-: track 0.00 -> 7.84 mm
- net /freq_converter/RF_CONN+: track 0.00 -> 7.83 mm
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Other:
- board text added: "ANT IN-"
- board text added: "Do not use"
- board text added: "IF_OUT-"
- board text added: "Rev. 2.3 | 2026-03-03"
- board text removed: "= OK"
- board text removed: "Only if antenna feed is on the left if not it'll probably work anyway"
- board text removed: "Rev. 2.2 | 2026-02-22"
- board text removed: "Traces under ESP? reroute so traces on module dont crosstalk?"
- board text removed: "https://docs.espressif.com/projects/esp-hardware-design-guidelines/en/latest/esp32c3/pcb-layout-design.html"
