File: Tesla_rev_2/f_conv.kicad_sch (KiCad schematic)
At the start: 32 parts, among them J8 Conn_01x02, J9 Conn_01x02, U8 AD831, Y1 OSC25M-3.3I/S5

Commit message: changes with BOM, minor fixes
Parts:
- L3: value 870nF -> 870nH
Changed lines of the file:
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@@
 			)
 		)
-		(property "Value" "870nF"
+		(property "Value" "870nH"
 			(at 180.975 82.55 90)
 			(effects

Commit message: Board ready for manufacturing, no more changes to either KiCad projects
Parts:
- removed C33: 470pF, Capacitor_SMD:C_0603_1608Metric, symbol Device:C
- removed C34: 220pF, Capacitor_SMD:C_0603_1608Metric, symbol Device:C
- removed C43: 2.2nF, Capacitor_SMD:C_0603_1608Metric, symbol Device:C_Small
- removed L5: TBD, Inductor_SMD:L_0603_1608Metric, symbol Device:L
- removed L6: 12nH, Inductor_SMD:L_0603_1608Metric, symbol Device:L
- removed L7: 20nH, Inductor_SMD:L_0603_1608Metric, symbol Device:L
- removed R29: 50, Capacitor_SMD:C_0805_2012Metric, symbol Device:R
- added C33: 100nF, Capacitor_SMD:C_0603_1608Metric, symbol Device:C_Small
- added C34: 5pF, Capacitor_SMD:C_0603_1608Metric, symbol Device:C_Small
- added L5: 430nH, Inductor_SMD:L_0603_1608Metric, symbol Device:L_Small
- added L6, L7: MABAES0060, Tesla_Library:SM-22, symbol Tesla_sextant_BT_Library:MABAES0060
- added R29: 200, Resistor_SMD:R_0805_2012Metric, symbol Device:R_Small
- added R34: 75, Resistor_SMD:R_0805_2012Metric, symbol Device:R
- C31: value 5.6pF -> 5pF
- C32: value 4.7pF -> 130pF
- C35: value TBD -> 5pF; footprint Capacitor_SMD:C_0805_2012Metric -> Capacitor_SMD:C_0603_1608Metric
- C36: value 100nF -> 510pF; footprint Capacitor_SMD:C_0805_2012Metric -> Capacitor_SMD:C_0603_1608Metric
- C39: value 2.2nF -> 44pF
- L3: value 870nH -> 1uH; footprint Inductor_SMD:L_0805_2012Metric -> Inductor_SMD:L_0603_1608Metric; Part_num DL0805-0.082 -> (none)
- L4: value 1.3uF -> 40nH; footprint Inductor_SMD:L_0805_2012Metric -> Inductor_SMD:L_0603_1608Metric; Part_num DL0805-1.2 -> (none)
- L8: value 18nH -> 900nH
- R27, R33: value 50 -> 75; footprint Capacitor_SMD:C_0805_2012Metric -> Resistor_SMD:R_0805_2012Metric
- R28, R30, R31, R32: footprint Capacitor_SMD:C_0805_2012Metric -> Resistor_SMD:R_0805_2012Metric
Connections:
- net IF_C3 is gone; now on net GND: C32.1, L4.2
- net GND: now also C36.2, C33.2, L5.2, L6.2, L6.5, L7.3, R34.2; no longer C35.1, C36.1, C39.1, J8.2 (Pin_2), J9.2 (Pin_2)
- net LO_LPF: now also C39.1
- net LO_OSC: now also R29.2; no longer L8.1
- net RF_IN-: now also C33.1; no longer C36.2
- net IF_C1 renamed IF_BPF
- net IF_BPF: now also C32.2, L4.1, L6.4, R34.1; no longer C31.2
- net IF_FLT renamed IF_C
- net IF_C: now also C31.2; no longer C32.2
- net IF_OUT renamed IF_OUT+
- net IF_OUT+: now also L6.1; no longer L4.1
- net IF_R1 renamed IF_TERM
- net LO_HPF renamed LO_L1
- net RF_CONN renamed RF_CONN+
- net RF_CONN+: now also L7.4
- new net: C36.1, L8.1, R29.1
- new net IF_OUT-: J8.2 (Pin_2), L6.3
- new net RF_CONN-: J9.2 (Pin_2), L7.5
- new net RF_T: C34.1, L7.1
- new net RF_Z: C34.2, C35.1, L5.1
- no-connect marks 1 -> 2
Other:
- note added: "2nd order chebyshev BPF fc = 70MHz, B= 10MHz"
- note added: "75 ohm coax"
- note added: "C39: Xc = 1/2 PI f C => C = 1/2 PI f Xc C = 1/(2 PI 25MHz 120 ohm)"
- note added: "Imax = 20mA"
- note added: "L8: Xl = 2 PI f L L = Xl / 2 PI f L = 120ohm / (2 PI 25MHz)"
- note added: "Umax +/- 1V"
- note removed: "65 - 75MHz Cheby. filter type 1, 4th order BPF"
- note removed: "R termination - AD831 DSH pg. 9 Driving filters"
- note removed: "Z-matching"
- moved on the sheet: C28, C29, C30, C37, C38, C39, C40, C42, J8, J9, L8, R27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

Commit message: Final Project Commit
Other:
- note added: "ADC"
- note added: "MCU"
- note added: "SW USB driver"
- note added: "USB-C"
