File: Front_Panel/Front_Panel.kicad_sch (KiCad schematic)
At the start: 27 parts, among them J2 Conn_01x05, Q1 BC817, SW1 SW_Push, SW2 SW_Push, SW3 SW_Push, SW4 SW_Push, U1 NHD-C0220BIZ, U2 MCP23008-xSO

Commit message: changes with BOM, minor fixes
Parts:
- added J2: Conn_01x05, Connector_PinSocket_2.00mm:PinSocket_1x05_P2.00mm_Vertical, symbol Connector_Generic:Conn_01x05
- J1: renamed from J2; footprint Connector_PinSocket_2.54mm:PinSocket_1x05_P2.54mm_Vertical -> Connector_PinSocket_2.00mm:PinSocket_1x05_P2.00mm_Vertical
- renumbered C7 to C2, C2 to C3, C3 to C4, C4 to C5, C5 to C6, C6 to C7
Connections:
- net +3.3V: now also J2.4 (Pin_4)
- net GND: now also J2.5 (Pin_5)
- net at U2.15 (GP5): now also J2.1 (Pin_1)
- net at U2.16 (GP6): now also J2.2 (Pin_2)
- net at U2.17 (GP7): now also J2.3 (Pin_3)
- no-connect marks 5 -> 2
Other:
- note added: "Breakout for unused pins"

Commit message: Final Project Commit
Connections:
- net +3.3V: now also U1.1 (~{RST}), U2.6 (~{RESET})
- no-connect marks 2 -> 0
